File: Z8S180_57Q.kicad_sch (KiCad schematic)
At the start: 22 parts, among them J1 Conn_01x06_Pin, J16 Conn_01x06_Pin, J2 Conn_01x05, J3 Barrel_Jack_Switch, J5 Conn_01x02, J5 Conn_01x08_Pin, SW1 SW_SPDT, SW2 SW_SPST, U1 Z8S180_68PLCC, U2 AS6C4008-55PCN, U3 PIC18F57Q43-IPT

Commit message: schematics complete. change README.md
Parts:
- removed J1, J16: Conn_01x06_Pin, 0-local:PinHeader_1x06_P2.54mm_Horizontal_NoFeet, symbol Connector:Conn_01x06_Pin
- removed J5: Conn_01x08_Pin, 0-local:PinHeader_1x08_P2.54mm_Rev_Horizontal_Nofoot, symbol Connector:Conn_01x08_Pin
- removed SW1: SW_SPDT, 0-local:PowerSW_for_SBC_series, symbol Switch:SW_SPDT
- added C1, C2: 20pF, symbol Device:C_Small
- added C5: 0.1uF, Capacitor_THT:C_Disc_D3.0mm_W2.0mm_P2.50mm, symbol Device:C_Small
- added D1: 1N4148, Diode_THT:D_DO-35_SOD27_P7.62mm_Horizontal, symbol Diode:1N4148
- added J1: SPI1, symbol Connector_Generic:Conn_01x06
- added J11: Conn_01x03, symbol 0-Project:Conn_01x03
- added J12: Conn_01x02, symbol 0-Project:Conn_01x02_trans
- added J13, J3: Conn_01x02, symbol Connector_Generic:Conn_01x02
- added J14: Power SW, symbol 0-Project:Conn_01x03
- added J16: PIC-Serial, symbol Connector_Generic:Conn_01x06
- added J4: SNAP, symbol Connector_Generic:Conn_01x08
- added J6: Z8S180-Serial, symbol Connector_Generic:Conn_01x06
- added JP1, JP2, JP4, JP5, JP6: Jumper_2_Open, symbol Jumper:Jumper_2_Open
- added JP3: Jumper_2_Bridged, symbol Jumper:Jumper_2_Bridged
- added R1, R3, R4, R5: 10k, Resistor_THT:R_Axial_DIN0204_L3.6mm_D1.6mm_P7.62mm_Horizontal, symbol Device:R
- added Y1: Crystal, symbol Device:Crystal_Small
- J2: value Conn_01x05 -> SPI2
- renumbered C2 to C4, C1 to C7, D1 to D2, D2 to D3, J5 to J15, J3 to J17, R5 to R6, R4 to R7, R1 to R8, R3 to R9, SW2 to SW1
Connections:
- net A17: now also JP6.1 (A), JP6.2 (B), R5.2
- net CLK: now also J11.3 (Pin_3), J12.1 (Pin_1)
- net GND: now also U1.56 (RXS/CTS1), C1.1, C2.1, C5.2, J1.6 (Pin_6), J16.6 (Pin_6), J4.3 (Pin_3), J6.6 (Pin_6), JP1.1 (A), JP2.1 (A), JP5.2 (B)
- net VCC: now also U1.11 (~{INT1}), U1.12 (~{INT2}), U1.58 (~{DREQ1}), C5.1, J1.5 (Pin_5), J14.3 (Pin_3), J4.2 (Pin_2), JP3.1 (A), JP4.2 (B), R1.1, R3.1, R4.1; no longer J15.1 (Pin_1)
- net ~{RD}: now also U2.29 (WE#); no longer U2.24 (OE#)
- net ~{WR}: now also U2.24 (OE#); no longer U2.29 (WE#)
- net at R2.2, SW1.1 (A), U3.20 (~{MCLR}): now also J4.1 (Pin_1)
- net at U3.33 (RA6): now also J16.2 (Pin_2)
- net at J2.5 (Pin_5), U3.34 (RC0): now also J1.2 (Pin_2)
- net at J2.3 (Pin_3), U3.35 (RC1): now also J1.3 (Pin_3)
- net at U3.40 (RC2): now also J1.4 (Pin_4)
- net at U3.41 (RC3): now also J2.4 (Pin_4)
- net at U3.46 (RC4): now also J1.1 (Pin_1); no longer J2.4 (Pin_4)
- net DC_POWER: now reaches J17.1
- net DC_POWER: now also J15.1 (Pin_1), J14.1 (Pin_1), J14.2 (Pin_2), J3.1 (Pin_1)
- net at D2.1 (K): now also J16.3 (Pin_3)
- net A18: now reaches R6.1, U1.33 (A18), U2.1 (A18)
- net A16: now reaches R7.1, U1.31 (A16), U2.2 (A16)
- net at J15.2 (Pin_2): now also J16.4 (Pin_4)
- net at U1.3 (XTAL): now also J13.1 (Pin_1)
- net at U1.46 (~{CTS0}): now also JP1.2 (B)
- net at U1.47 (~{DCD0}): now also JP2.2 (B)
- net at U1.48 (TXA0): now also J6.2 (Pin_2)
- net at U1.49 (RXA0): now also D1.2 (A), R1.2
- net at U1.50 (CKA0/~{DREQ0}): now also U1.54 (CKA1/~{TEND0}), J12.2 (Pin_2), R4.2
- net at U1.53 (RXA1): now also JP3.2 (B)
- net at U1.9 (~{NMI}): now also R3.2
- net A6 renamed A6/PGC
- net A6/PGC: now also J4.5 (Pin_5)
- net A7 renamed A7/PGD
- net A7/PGD: now also J4.4 (Pin_4)
- new net: D1.1 (K), J6.3 (Pin_3)
- new net: J3.2 (Pin_2), J6.4 (Pin_4)
- new net: C1.2, J11.1 (Pin_1), Y1.2
- new net: J11.2 (Pin_2), U1.5 (~{WAIT})
- new net: JP4.1 (A), JP5.1 (A), R5.1
- new net: C2.2, J13.2 (Pin_2), Y1.1
- no-connect marks 9 -> 19
Other:
- note added: "CLK"
- note added: "CS1"
- note added: "CS2"
- note added: "DIN"
- note removed: "CS"
- moved on the sheet: C3, C4, C6, C7, D3, J17, J2, R6, R7, R9, U2, U3
